Commit message: feat: add RGBD deep camera to the robot

File: src/my_robot/urdf/my_robot.xacro (robot description, xacro)
@@ -46,5 +46,5 @@
 	<!-- wheels -->
   <joint type="continuous" name="left_front_wheel_hinge">
-    <origin xyz="0.15 0.15 0" rpy="0 0 0"/>
+    <origin xyz="0.15 0.16 0" rpy="0 0 0"/>
     <child link="left_front_wheel"/>
     <parent link="chassis"/>
@@ -87,5 +87,5 @@
 	</link>
   <joint type="continuous" name="right_front_wheel_hinge">
-    <origin xyz="0.15 -0.15 0" rpy="0 0 0"/>
+    <origin xyz="0.15 -0.16 0" rpy="0 0 0"/>
     <child link="right_front_wheel"/>
     <parent link="chassis"/>
@@ -128,5 +128,5 @@
 	</link>
   <joint type="continuous" name="left_back_wheel_hinge">
-    <origin xyz="-0.15 0.15 0" rpy="0 0 0"/>
+    <origin xyz="-0.15 0.16 0" rpy="0 0 0"/>
     <child link="left_back_wheel"/>
     <parent link="chassis"/>
@@ -169,5 +169,5 @@
 	</link>
   <joint type="continuous" name="right_back_wheel_hinge">
-    <origin xyz="-0.15 -0.15 0" rpy="0 0 0"/>
+    <origin xyz="-0.15 -0.16 0" rpy="0 0 0"/>
     <child link="right_back_wheel"/>
     <parent link="chassis"/>
@@ -209,7 +209,7 @@
     </inertial>
 	</link>
-	<!-- sensors -->
+	<!-- RGBD CAMERA SENSOR -->
   <joint type="fixed" name="camera_joint">
-    <origin xyz="0.275 0 0.045" rpy="0 0 0"/>
+    <origin xyz="0.275 0.075 0.045" rpy="0 0 0"/>
     <child link="camera"/>
     <parent link="chassis"/>
@@ -239,4 +239,34 @@
     </inertial>
 	</link>
+  <joint name="camera_optical_joint" type="fixed">
+    <origin xyz="0 -0.15 0" rpy="0 0 0"/>
+    <parent link="camera"/>
+    <child link="camera_optical"/>
+    <axis xyz="0 1 0" rpy="0 0 0"/>
+  </joint>
+  <link name="camera_optical">
+    <collision name='camera_optical_collision'>
+      <origin xyz="0 0 0" rpy=" 0 0 0"/>
+      <geometry>
+        <box size="0.05 0.05 0.05"/>
+      </geometry>
+    </collision>
+    <visual name='camera_optical_visual'>
+      <origin xyz="0 0 0" rpy=" 0 0 0"/>
+      <geometry>
+        <box size="0.05 0.05 0.05"/>
+      </geometry>
+    </visual>
+    <inertial>
+      <mass value="0.1"/>
+      <origin xyz="0.0 0 0" rpy=" 0 0 0"/>
+      <inertia
+          ixx="1e-6" ixy="0" ixz="0"
+          iyy="0.000001" iyz="0"
+          izz="0.000001"
+      />
+    </inertial>
+  </link>
+	<!-- LASER SENSOR -->
   <joint type="fixed" name="hokuyo_joint">
     <origin xyz="0.275 0 -0.055" rpy="0 0 0"/>

Commit message: fix: robot second camera pose and depth camera plugin configuration

File: src/my_robot/urdf/my_robot.xacro (robot description, xacro)
@@ -211,5 +211,5 @@
 	<!-- RGBD CAMERA SENSOR -->
   <joint type="fixed" name="camera_joint">
-    <origin xyz="0.275 0.075 0.045" rpy="0 0 0"/>
+    <origin xyz="0.275 0.0 0.045" rpy="0 0 0"/>
     <child link="camera"/>
     <parent link="chassis"/>
@@ -240,8 +240,8 @@
 	</link>
   <joint name="camera_optical_joint" type="fixed">
-    <origin xyz="0 -0.15 0" rpy="0 0 0"/>
+    <origin xyz="0 0 0" rpy="-1.5707 0 -1.5707"/>
     <parent link="camera"/>
     <child link="camera_optical"/>
-    <axis xyz="0 1 0" rpy="0 0 0"/>
+    <axis xyz="0 0 0" rpy="0 0 0"/>
   </joint>
   <link name="camera_optical">
